File: PCB/mycoolpad.kicad_pcb (KiCad board)
At the start: 2 copper layers, 67.2 x 91.1 mm, 30 parts, among them J1 Conn_01x04, SW1 SW_Push, SW10 RotaryEncoder_Switch, SW2 SW_Push, SW3 SW_Push, SW4 SW_Push, SW5 SW_Push, SW6 SW_Push, SW7 SW_Push, SW8 SW_Push, SW9 SW_Push, U1 XIAO-RP2040-DIP

Commit message: Add files via upload
Parts:
- moved J1 5.54 mm to (124.8, 58.1)
- moved SW10 4.85 mm to (161.7, 52.0)
Routing:
- net /ENC_A: track 33.6 -> 38.3 mm
- net /ENC_B: track 35.5 -> 39.2 mm
- net /ROW1: track 83.9 -> 80.8 mm
- net /COL1: track 115.6 -> 113.3 mm
- net +3.3V: track 27.7 -> 29.8 mm
- net /OLED_SCL: track 8.35 -> 9.76 mm
- net +5V: track 326.1 -> 327.1 mm
- net /OLED_SDA: track 9.18 -> 9.76 mm
Changed lines of the file:
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@@
 	(footprint "Connector_PinHeader_2.54mm:PinHeader_1x04_P2.54mm_Vertical"
 		(layer "F.Cu")
-		(at 124.32 52.58 180)
+		(at 124.79 58.1 180)
 		(descr "Through hole straight pin header, 1x04, 2.54mm pitch, single row")
 		(tags "Through hole pin header THT 1x04 2.54mm single row")
@@
 	(footprint "Rotary_Encoder:RotaryEncoder_Alps_EC11E-Switch_Vertical_H20mm"
 		(layer "F.Cu")
-		(at 161.97 47.17)
+		(at 161.68 52.01)
 		(descr "Alps rotary encoder, EC11E... with switch, vertical shaft, http://www.alps.com/prod/info/E/HTML/Encoder/Incremental/EC11/EC11E15204A3.html")
 		(tags "rotary encoder")
@@
 		)
 		(fp_text user "${REFERENCE}"
-			(at 11.1 6.3 0)
+			(at 4.36 -0.05 0)
 			(layer "F.Fab")
 			(effects
@@
 	)
 	(segment
-		(start 174.581 52.381)
-		(end 174.581 76.247686)
+		(start 160.05 36.3)
+		(end 174.581 50.831)
 		(width 0.2)
 		(layer "F.Cu")
@@
 	)
 	(segment
-		(start 162.009 100.229)
-		(end 163.18 101.4)
+		(start 148.12 36.3)
+		(end 160.05 36.3)
 		(width 0.2)
 		(layer "F.Cu")
@@
 	)
 	(segment
-		(start 148.12 36.3)
-		(end 158.5 36.3)
+		(start 162.009 100.229)
+		(end 163.18 101.4)
 		(width 0.2)
 		(layer "F.Cu")
@@
 	)
 	(segment
-		(start 174.581 76.247686)
-		(end 171.004343 79.824343)
+		(start 174.581 50.831)
+		(end 174.581 76.247686)
 		(width 0.2)
 		(layer "F.Cu")
@@
 	)
 	(segment
-		(start 158.5 36.3)
-		(end 174.581 52.381)
+		(start 162.009 88.819686)
+		(end 162.009 100.229)
 		(width 0.2)
 		(layer "F.Cu")
@@
 	)
 	(segment
-		(start 162.009 88.819686)
-		(end 162.009 100.229)
+		(start 174.581 76.247686)
+		(end 171.004343 79.824343)
 		(width 0.2)
 		(layer "F.Cu")
@@
 	)
 	(segment
+		(start 129.72224 43.92)
+		(end 132.88 43.92)
+		(width 0.2)
+		(layer "F.Cu")
+		(net 2)
+	)
+	(segment
+		(start 119.21 54.42)
+		(end 120.63776 52.99224)
+		(width 0.2)
+		(layer "F.Cu")
+		(net 2)
+	)
+	(segment
 		(start 120.7527 94.9148)
 		(end 121.8837 93.7838)
@@
 	)
 	(segment
-		(start 120.18 73.7301)
-		(end 120.18 47.47224)
-		(width 0.2)
-		(layer "F.Cu")
-		(net 2)
-	)
-	(segment
 		(start 120.7827 92.6828)
 		(end 120.7827 76.4748)
@@
 	)
 	(segment
-		(start 121.8537 75.4038)
-		(end 120.18 73.7301)
+		(start 119.21 72.7601)
+		(end 119.21 54.42)
 		(width 0.2)
 		(layer "F.Cu")
@@
 	)
 	(segment
-		(start 120.18 47.47224)
-		(end 125.13224 42.52)
+		(start 120.65 52.99224)
+		(end 129.72224 43.92)
 		(width 0.2)
 		(layer "F.Cu")
@@
 	)
 	(segment
-		(start 132.045 43.92)
-		(end 132.88 43.92)
+		(start 120.63776 52.99224)
+		(end 120.65 52.99224)
 		(width 0.2)
 		(layer "F.Cu")
@@
 	)
 	(segment
-		(start 125.13224 42.52)
-		(end 130.645 42.52)
+		(start 132.045 43.92)
+		(end 132.88 43.92)
 		(width 0.2)
 		(layer "F.Cu")
@@
 	)
 	(segment
-		(start 130.645 42.52)
-		(end 132.045 43.92)
+		(start 121.8537 113.4738)
+		(end 120.7527 112.3728)
 		(width 0.2)
 		(layer "F.Cu")
@@
 	)
 	(segment
-		(start 121.8537 113.4738)
-		(end 120.7527 112.3728)
+		(start 121.8537 75.4038)
+		(end 119.21 72.7601)
 		(width 0.2)
 		(layer "F.Cu")
@@
 	)
 	(segment
-		(start 124.32 44.96)
-		(end 125.82 46.46)
+		(start 128.81 46.46)
+		(end 132.88 46.46)
 		(width 0.2)
 		(layer "F.Cu")
@@
 	)
 	(segment
-		(start 125.82 46.46)
-		(end 132.88 46.46)
+		(start 124.79 50.48)
+		(end 128.81 46.46)
 		(width 0.2)
 		(layer "F.Cu")
@@
 	)
 	(segment
-		(start 124.32 50.04)
-		(end 124.757 50.477)
+		(start 129.873 50.477)
+		(end 139.023 50.477)
 		(width 0.2)
 		(layer "F.Cu")
@@
 	)
 	(segment
-		(start 124.757 50.477)
-		(end 139.023 50.477)
+		(start 124.79 55.56)
+		(end 125.227 55.997)
 		(width 0.2)
 		(layer "F.Cu")
@@
 	)
 	(segment
-		(start 125.82 49)
-		(end 132.045 49)
+		(start 124.79 55.56)
+		(end 129.873 50.477)
 		(width 0.2)
 		(layer "F.Cu")
-		(net 25)
+		(net 24)
 	)
 	(segment
-		(start 124.32 47.5)
-		(end 125.82 49)
+		(start 124.79 53.02)
+		(end 128.81 49)
 		(width 0.2)
 		(layer "F.Cu")
@@
 	)
 	(segment
-		(start 132.71 66.76)
-		(end 132.71 64.41)
+		(start 128.81 49)
+		(end 132.88 49)
 		(width 0.2)
 		(layer "F.Cu")
-		(net 26)
+		(net 25)
 	)
 	(segment
-		(start 156.960108 49)
-		(end 170.84 62.879892)
+		(start 132.71 66.76)
+		(end 132.71 64.41)
 		(width 0.2)
 		(layer "F.Cu")
@@
 	)
 	(segment
-		(start 170.84 62.879892)
-		(end 170.84 66.76)
+		(start 148.12 49)
+		(end 149.42 49)
 		(width 0.2)
 		(layer "F.Cu")
@@
 	)
 	(segment
-		(start 148.12 49)
-		(end 156.960108 49)
+		(start 145.74 51.38)
+		(end 148.12 49)
 		(width 0.2)
 		(layer "F.Cu")
@@
 	)
 	(segment
-		(start 145.74 51.38)
-		(end 148.12 49)
+		(start 151.76 104.84)
+		(end 155.521 101.079)
 		(width 0.2)
 		(layer "F.Cu")
@@
 	)
 	(segment
-		(start 151.76 104.84)
-		(end 155.521 101.079)
+		(start 167.18 66.76)
+		(end 170.84 66.76)
+		(width 0.2)
+		(layer "F.Cu")
+		(net 26)
+	)
+	(segment
+		(start 149.42 49)
+		(end 167.18 66.76)
 		(width 0.2)
 		(layer "F.Cu")
@@
 	)
 	(segment
-		(start 160.7 52.17)
-		(end 150.472 41.942)
+		(start 160.379 55.709)
+		(end 161.68 57.01)
 		(width 0.2)
 		(layer "F.Cu")
@@
 	)
 	(segment
-		(start 150.472 41.942)
-		(end 150.472 40.578374)
-		(width 0.2)
-		(layer "F.Cu")
-		(net 29)
-	)
-	(segment
-		(start 133.16 41.66)
-		(end 132.88 41.38)
-		(width 0.2)
-		(layer "F.Cu")
-		(net 29)
-	)
-	(segment
-		(start 146.33669 41.66)
-		(end 133.16 41.66)
+		(start 133.943 40.317)
+		(end 150.210626 40.317)
 		(width 0.2)
 		(layer "F.Cu")
@@
 	(segment
 		(start 150.210626 40.317)
-		(end 147.67969 40.317)
+		(end 160.379 50.485374)
 		(width 0.2)
 		(layer "F.Cu")
@@
 	)
 	(segment
-		(start 147.67969 40.317)
-		(end 146.33669 41.66)
+		(start 160.379 50.485374)
+		(end 160.379 55.709)
 		(width 0.2)
 		(layer "F.Cu")
@@
 	)
 	(segment
-		(start 150.472 40.578374)
-		(end 150.210626 40.317)
+		(start 132.88 41.38)
+		(end 133.943 40.317)
 		(width 0.2)
 		(layer "F.Cu")
@@
 	)
 	(segment
-		(start 161.97 52.17)
-		(end 160.7 52.17)
+		(start 133.11 39.07)
+		(end 143.84669 39.07)
 		(width 0.2)
-		(layer "F.Cu")
-		(net 29)
+		(layer "B.Cu")
+		(net 31)
 	)
 	(segment
-		(start 148.57331 37.79)
-		(end 152.59 37.79)
+		(start 147.67969 37.777)
+		(end 148.56031 37.777)
 		(width 0.2)
 		(layer "B.Cu")
@@
 	)
 	(segment
-		(start 147.66669 37.79)
-		(end 147.67969 37.777)
+		(start 143.84669 39.07)
+		(end 145.12669 37.79)
 		(width 0.2)
 		(layer "B.Cu")
@@
 	)
 	(segment
-		(start 145.12669 37.79)
-		(end 147.66669 37.79)
+		(start 132.88 38.84)
+		(end 133.11 39.07)
 		(width 0.2)
 		(layer "B.Cu")
@@
 	)
 	(segment
-		(start 143.84669 39.07)
-		(end 145.12669 37.79)
+		(start 148.57331 37.79)
+		(end 152.59 37.79)
 		(width 0.2)
 		(layer "B.Cu")
@@
 	)
 	(segment
-		(start 147.67969 37.777)
-		(end 148.56031 37.777)
+		(start 145.12669 37.79)
+		(end 147.66669 37.79)
 		(width 0.2)
 		(layer "B.Cu")
@@
 	)
 	(segment
-		(start 132.88 38.84)
-		(end 133.11 39.07)
+		(start 161.68 46.88)
+		(end 161.68 52.01)
 		(width 0.2)
 		(layer "B.Cu")
@@
 	)
 	(segment
-		(start 133.11 39.07)
-		(end 143.84669 39.07)
+		(start 152.59 37.79)
+		(end 161.68 46.88)
 		(width 0.2)
 		(layer "B.Cu")
@@
 	)
 	(segment
-		(start 152.59 37.79)
-		(end 161.97 47.17)
+		(start 147.66669 37.79)
+		(end 147.67969 37.777)
 		(width 0.2)
 		(layer "B.Cu")
